Commit message: remove collision tag from semantic/symbolic ee_link that added a random cube that was causing problems, is now just a virtual link for adding other components/measuring distance as it should be

File: armada_description/universal_robot/urdf/ur5e.urdf.xacro (robot description, xacro)
@@ -325,10 +325,4 @@
     </joint>
     <link name="${prefix}ee_link">
-      <collision>
-        <geometry>
-          <box size="0.01 0.01 0.01"/>
-        </geometry>
-        <origin rpy="0 0 0" xyz="-0.01 0 0"/>
-      </collision>
     </link>
     <xacro:ur_arm_transmission prefix="${prefix}" />

Commit message: add parameter 'parent' and joint to connect base_link to parent in ur5e description, apply parameter in robot_description xacro files for robot bringup

File: armada_description/universal_robot/urdf/ur5e.urdf.xacro (robot description, xacro)
@@ -12,5 +12,5 @@
     </inertial>
   </xacro:macro>
-  <xacro:macro name="ur5e_robot" params="prefix joint_limited
+  <xacro:macro name="ur5e_robot" params="prefix joint_limited parent
     shoulder_pan_lower_limit:=${-pi}    shoulder_pan_upper_limit:=${pi}
     shoulder_lift_lower_limit:=${-pi}    shoulder_lift_upper_limit:=${pi}
@@ -77,4 +77,13 @@
     <xacro:property name="forearm_radius" value="0.040" />    <!-- manually measured -->
     <xacro:property name="wrist_radius" value="0.045" />      <!-- manually measured -->
+    <!-- <link name="world" /> -->
+    <joint name="${prefix}base_link_joint" type="fixed">
+        <parent link="${parent}"/>
+        <child link="base_link"/>
+        <origin rpy="0 0 0" xyz="0 0 0"/>
+        <!-- for simulation -->
+        <dynamics damping="1.0"/>
+        <!-- end for simulation -->
+      </joint>
     <link name="${prefix}base_link" >
       <visual>

File: armada_description/universal_robot/urdf/ur5e_robot_d435_millibar_r2f85.urdf.xacro (robot description, xacro)
@@ -12,5 +12,5 @@
   <xacro:include filename="$(find armada_gazebo)/robotiq/urdf/robotiq_2f_85_transmission_macro.xacro" />
   <!-- arm -->
-  <xacro:ur5e_robot prefix="" joint_limited="false" />
+  <xacro:ur5e_robot prefix="" joint_limited="false" parent="world"/>
   <!-- camera mount/millibar stuff -->
   <xacro:load_d435_millibar parent="ee_link" prefix="" />
@@ -19,10 +19,3 @@
   <xacro:load_gazebo_gripper_transmissions prefix=""/>
   <link name="world" />
-  <joint name="connect_world_and_base_link" type="fixed">
-    <child link="world" />
-    <parent link="base_link" />
-    <origin xyz="0.0 0.0 0.0" rpy="0.0 0.0 0.0" />
-    <!-- <origin xyz="0.0 0.0 0.41" rpy="0.0 0.0 0.0" /> -->
-    <!-- <origin xyz="0.0 0.0 0.00475" rpy="0.0 0.0 ${pi/2}" /> -->
-  </joint>
 </robot>

File: armada_description/universal_robot/urdf/ur5e_robot_d435_millibar_r2f85_workstation.urdf.xacro (robot description, xacro)
@@ -14,5 +14,5 @@
   <xacro:include filename="$(find armada_gazebo)/robotiq/urdf/robotiq_2f_85_transmission_macro.xacro" />
   <!-- arm -->
-  <xacro:ur5e_robot prefix="" joint_limited="false" />
+  <xacro:ur5e_robot prefix="" joint_limited="false" parent="world"/>
   <!-- camera mount/millibar stuff -->
   <xacro:load_d435_millibar parent="ee_link" prefix="" />
