Commit message: delete unused description files and those with old workstation style; no longer spawning as part of robot urdf, add joint limited version of typical description

File: armada_description/universal_robot/urdf/ur5e_joint_limited_robot_d435_millibar_r2f85.urdf.xacro (robot description, xacro)
@@ -6,6 +6,4 @@
   <!-- ur5e -->
   <xacro:include filename="$(find armada_description)/universal_robot/urdf/ur5e.urdf.xacro" />
-  <!-- ARMada workstation -->
-  <xacro:include filename="$(find armada_description)/armada_test_station/urdf/workstation_model.urdf.xacro" />
   <!-- realsense d435i mount + millibar (robot & gripper side) adapters -->
   <xacro:include filename="$(find armada_description)/armada_tooling/urdf/d435_millibar_macro.urdf.xacro" />
@@ -14,23 +12,15 @@
   <xacro:include filename="$(find armada_gazebo)/robotiq/urdf/robotiq_2f_85_transmission_macro.xacro" />
   <!-- arm -->
-  <xacro:ur5e_robot prefix="" joint_limited="false" parent="world"/>
-  <!-- camera mount/millibar stuff -->
-  <xacro:load_d435_millibar parent="ee_link" prefix="" />
+  <xacro:ur5e_robot prefix="" joint_limited="true" parent="world"
+    shoulder_pan_lower_limit="${-pi}" shoulder_pan_upper_limit="${pi}"
+    shoulder_lift_lower_limit="${-pi}" shoulder_lift_upper_limit="${pi}"
+    elbow_joint_lower_limit="${-pi}" elbow_joint_upper_limit="${pi}"
+    wrist_1_lower_limit="${-pi}" wrist_1_upper_limit="${pi}"
+    wrist_2_lower_limit="${-pi}" wrist_2_upper_limit="${pi}"
+    wrist_3_lower_limit="${-pi}" wrist_3_upper_limit="${pi}"
+  />
   <!-- gripper -->
   <xacro:load_gripper parent="tooling_ee_link"  prefix=""/>
   <xacro:load_gazebo_gripper_transmissions prefix=""/>
-  <!-- workstation -->
-  <xacro:workstation prefix="table_" namespace=""/>
   <link name="world" />
-  <joint name="connect_world_and_table" type="fixed">
-    <child link="table_base_link" />
-    <parent link="world" />
-    <origin xyz="0.0 0.0 0.41" rpy="0.0 0.0 0.0" />
-  </joint>
-  <joint name="connect_table_and_arm" type="fixed">
-    <parent link="table_mounting_plate_link" />
-    <child link = "base_link" />
-    <!-- <origin xyz="0.0 0.0 0.03625" rpy="0.0 0.0 ${pi/2}" /> -->
-    <origin xyz="0.0 0.0 0.00475" rpy="0.0 0.0 ${pi/2}" />
-  </joint>
 </robot>

File: armada_description/universal_robot/urdf/ur5e_robot.urdf.xacro (robot description, xacro)
@@ -7,10 +7,5 @@
   <xacro:include filename="$(find armada_description)/universal_robot/urdf/ur5e.urdf.xacro" />
   <!-- arm -->
-  <xacro:ur5e_robot prefix="" joint_limited="false"/>
+  <xacro:ur5e_robot prefix="" joint_limited="false" parent="world"/>
   <link name="world" />
-  <joint name="world_joint" type="fixed">
-    <parent link="world" />
-    <child link = "base_link" />
-    <origin xyz="0.0 0.0 0.0" rpy="0.0 0.0 0.0" />
-  </joint>
 </robot>

File: armada_description/universal_robot/urdf/ur5e_robot_r2f85.urdf.xacro (robot description, xacro)
@@ -10,13 +10,8 @@
   <xacro:include filename="$(find armada_gazebo)/robotiq/urdf/robotiq_2f_85_transmission_macro.xacro" />
   <!-- arm -->
-  <xacro:ur5e_robot prefix="" joint_limited="false"/>
+  <xacro:ur5e_robot prefix="" joint_limited="false" parent="world"/>
   <!-- gripper -->
   <xacro:load_gripper parent="ee_link"  prefix=""/>
   <xacro:load_gazebo_gripper_transmissions prefix=""/>
   <link name="world" />
-  <joint name="world_joint" type="fixed">
-    <parent link="world" />
-    <child link = "base_link" />
-    <origin xyz="0.0 0.0 0.0" rpy="0.0 0.0 0.0" />
-  </joint>
 </robot>
