Commit message: rotate tool_frame origin to match previously used tcp_link dummy link for grasp planning math, consistent with orientation that has been working (old values commented)

File: armada_description/robotiq/urdf/robotiq_arg2f_85_model_macro.xacro (robot description, xacro)
@@ -184,5 +184,6 @@
     <link name="${prefix}tool_frame"/>
     <joint name="${prefix}tool_frame_joint" type="fixed">
-        <origin xyz="0 0 0.120" rpy="${pi/2} 0 ${pi/2}" />
+        <!-- <origin xyz="0 0 0.120" rpy="${pi/2} 0 ${pi/2}" /> -->
+        <origin xyz="0 0 0.120" rpy="0 0 0" />
         <parent link="${parent}" />
         <child link="${prefix}tool_frame" />
