Commit message: add/edit: tm5-700 moveit config remade, updated to follow known working style | ezgripper support files added and modified for use in robot descriptions; structure, gazebo etc.

File: armada_description/armada_tooling/urdf/d435_millibar_model_macro.urdf.xacro (robot description, xacro)
@@ -82,9 +82,4 @@
     <origin xyz="0.0 0.0 0.0" rpy="-${pi/2} -${pi/2} 0.0"/>
    </joint>
-  <!-- USE GROUPS INSTEAD, XACRO DOES NOT SEEM TO LIKE THIS METHOD (PREFIX NOT DEFINED ERROR)
-  <child unless="$(eval prefix == '')" link="${namespace}/${prefix}rear_optical" />
-  <child if="$(eval prefix == '')" link="${prefix}rear_optical" />
-  <link unless="$(eval prefix == '')" name="${namespace}/${prefix}rear_optical" />
-  -->
   <link name="${prefix}wrist_optical" />
   <joint name="${prefix}d435_to_wrist_optical_joint" type="fixed">

File: armada_description/sakerobotics/urdf/ezgripper_dual_gen2_articulated_model_macro.xacro (robot description, xacro)
@@ -6,4 +6,5 @@
         <origin xyz="0 0 0" rpy="0 0 0"/>
         <geometry>
+          <!-- <mesh filename="package://armada_description/sakerobotics/meshes/SAKE_Palm_Dual_Gen2.dae" scale="1 1 1"/>  -->
           <mesh filename="package://ezgripper_driver/meshes/ezgripper_gen2/SAKE_Palm_Dual_Gen2.stl"/>
         </geometry>
@@ -12,10 +13,12 @@
         <origin xyz="0 0 0" rpy="0 0 0"/>
         <geometry>
-          <mesh filename="package://ezgripper_driver/meshes/ezgripper_gen2/SAKE_Palm_Dual_Gen2.stl"/>
+          <!-- <mesh filename="package://armada_description/sakerobotics/meshes/SAKE_Palm_Dual_Gen2.dae" scale="1 1 1"/>  -->
+          <mesh filename="package://ezgripper_driver/meshes/ezgripper_gen2/SAKE_Palm_Dual_Gen2.stl"/> -->
         </geometry>
       </collision>
       <inertial>
-        <mass value=".3"/>
-        <inertia ixx="0.01" ixy="0.0" ixz="0.0" iyy="0.01" iyz="0.0" izz="0.01"/>
+        <origin xyz="0 0 1" rpy="0 0 0" />
+        <mass value="1" />
+        <inertia ixx="1" ixy="0" ixz="0" iyy="1" iyz="0" izz="1" />
       </inertial>
     </link>
@@ -44,5 +47,6 @@
         <origin xyz="0 0 0" rpy="0 0 0"/>
         <geometry>
-          <mesh filename="package://ezgripper_driver/meshes/ezgripper_gen2/SAKE_Finger_L1_Gen2.stl"/>
+          <!-- <mesh filename="package://armada_description/sakerobotics/meshes/SAKE_Finger_L1_Gen2.dae" scale="1 1 1"/>  -->
+          <mesh filename="package://ezgripper_driver/meshes/ezgripper_gen2/SAKE_Finger_L1_Gen2.stl"/> -->
         </geometry>
       </visual>
@@ -50,10 +54,12 @@
         <origin xyz="0 0 0" rpy="0 0 0"/>
         <geometry>
-          <mesh filename="package://ezgripper_driver/meshes/ezgripper_gen2/SAKE_Finger_L1_Gen2.stl"/>
+          <!-- <mesh filename="package://armada_description/sakerobotics/meshes/SAKE_Finger_L1_Gen2.dae" scale="1 1 1"/>  -->
+          <mesh filename="package://ezgripper_driver/meshes/ezgripper_gen2/SAKE_Finger_L1_Gen2.stl"/> -->
         </geometry>
       </collision>
       <inertial>
-        <mass value=".025"/>
-        <inertia ixx="0.01" ixy="0.0" ixz="0.0" iyy="0.01" iyz="0.0" izz="0.01"/>
+        <origin xyz="0 0 1" rpy="0 0 0" />
+        <mass value="1" />
+        <inertia ixx="1" ixy="0" ixz="0" iyy="1" iyz="0" izz="1" />
       </inertial>
     </link>
@@ -64,4 +70,5 @@
         <origin xyz="0 0 0" rpy="0 0 0"/>
         <geometry>
+          <!-- <mesh filename="package://armada_description/sakerobotics/meshes/SAKE_Finger_L2_Gen2.dae" scale="1 1 1"/>  -->
           <mesh filename="package://ezgripper_driver/meshes/ezgripper_gen2/SAKE_Finger_L2_Gen2.stl"/>
         </geometry>
@@ -70,10 +77,12 @@
         <origin xyz="0 0 0" rpy="0 0 0"/>
         <geometry>
+          <!-- <mesh filename="package://armada_description/sakerobotics/meshes/SAKE_Finger_L2_Gen2.dae" scale="1 1 1"/>  -->
           <mesh filename="package://ezgripper_driver/meshes/ezgripper_gen2/SAKE_Finger_L2_Gen2.stl"/>
         </geometry>
       </collision>
       <inertial>
-        <mass value=".025"/>
-        <inertia ixx="0.01" ixy="0.0" ixz="0.0" iyy="0.01" iyz="0.0" izz="0.01"/>
+        <origin xyz="0 0 1" rpy="0 0 0" />
+        <mass value="1" />
+        <inertia ixx="1" ixy="0" ixz="0" iyy="1" iyz="0" izz="1" />
       </inertial>
     </link>
@@ -93,14 +102,9 @@
   </xacro:macro>
   <xacro:macro name="ezgripper_knuckle_L1_L2" params="prefix postfix reflectY reflectZ reflectR mimic_test">
-    <joint name="${prefix}_ezgripper_knuckle_L1_L2_${postfix}" type="revolute">
+    <joint name="${prefix}_ezgripper_knuckle_L1_L2_${postfix}" type="fixed">
       <parent link="${prefix}_ezgripper_finger_L1_${postfix}"/>
       <child link="${prefix}_ezgripper_finger_L2_${postfix}"/>
       <origin xyz="0.052 0 0" rpy="0 0 0"/>
-      <!-- origin xyz="0.06 0 0" rpy="${3.14159 * reflectR} 0 0"/-->
-      <axis xyz="0 1 0"/>
-      <limit lower="0" upper="1.94" effort="1" velocity="3.67"/>
-      <xacro:if value="${mimic_test}">
-           <mimic joint="${prefix}_ezgripper_knuckle_L1_L2_1"/>
-      </xacro:if>
+      <axis xyz="0 0 0"/>
     </joint>
   </xacro:macro>

File: armada_gazebo/robotiq/urdf/robotiq_2f_85_transmission_macro.xacro (robot description, xacro)
@@ -13,5 +13,6 @@
         </transmission>
         <gazebo>
-            <plugin filename="libroboticsgroup_gazebo_mimic_joint_plugin.so" name="mimic_robotiq_85_1">
+            <!-- <plugin filename="libroboticsgroup_gazebo_mimic_joint_plugin.so" name="mimic_robotiq_85_1"> -->
+            <plugin filename="libroboticsgroup_upatras_gazebo_mimic_joint_plugin.so" name="mimic_robotiq_85_1">
                 <joint>${prefix}finger_joint</joint>
                 <mimicJoint>${prefix}right_outer_knuckle_joint</mimicJoint>
@@ -21,5 +22,5 @@
                 <hasPID/>
             </plugin>
-            <plugin filename="libroboticsgroup_gazebo_mimic_joint_plugin.so" name="mimic_robotiq_85_2">
+            <plugin filename="libroboticsgroup_upatras_gazebo_mimic_joint_plugin.so" name="mimic_robotiq_85_2">
                 <joint>${prefix}finger_joint</joint>
                 <mimicJoint>${prefix}right_inner_knuckle_joint</mimicJoint>
@@ -29,5 +30,5 @@
                 <hasPID/>
             </plugin>
-            <plugin filename="libroboticsgroup_gazebo_mimic_joint_plugin.so" name="mimic_robotiq_85_3">
+            <plugin filename="libroboticsgroup_upatras_gazebo_mimic_joint_plugin.so" name="mimic_robotiq_85_3">
                 <joint>${prefix}finger_joint</joint>
                 <mimicJoint>${prefix}left_inner_knuckle_joint</mimicJoint>
@@ -37,5 +38,5 @@
                 <hasPID/>
             </plugin>
-            <plugin filename="libroboticsgroup_gazebo_mimic_joint_plugin.so" name="mimic_robotiq_85_4">
+            <plugin filename="libroboticsgroup_upatras_gazebo_mimic_joint_plugin.so" name="mimic_robotiq_85_4">
                 <joint>${prefix}finger_joint</joint>
                 <mimicJoint>${prefix}left_inner_finger_joint</mimicJoint>
@@ -45,5 +46,5 @@
                 <hasPID/>
             </plugin>
-            <plugin filename="libroboticsgroup_gazebo_mimic_joint_plugin.so" name="mimic_robotiq_85_5">
+            <plugin filename="libroboticsgroup_upatras_gazebo_mimic_joint_plugin.so" name="mimic_robotiq_85_5">
                 <joint>${prefix}finger_joint</joint>
                 <mimicJoint>${prefix}right_inner_finger_joint</mimicJoint>

File: armada_gazebo/sakerobotics/urdf/ezgripper_dual_gen2_transmission_macro.xacro (robot description, xacro)
@@ -21,4 +21,5 @@
         <hasPID/>
       </plugin>
+      <!--
       <plugin filename="libroboticsgroup_gazebo_mimic_joint_plugin.so" name="mimic_ezgripper_l1_l2_2">
         <joint>${prefix}_ezgripper_knuckle_L1_L2_1</joint>
@@ -29,4 +30,5 @@
         <hasPID/>
       </plugin>
+      -->
       <plugin name="gazebo_grasp_fix" filename="libgazebo_grasp_fix.so">
         <arm>

Commit message: switch .dae files back to .STL since STL is working and dae was not, confirm that collision is actually showing up and active in robot model (checked with rviz motion planning scene and moveit setup assistant for certainty)

File: armada_description/armada_tooling/urdf/d435_millibar_model_macro.urdf.xacro (robot description, xacro)
@@ -38,5 +38,5 @@
       <geometry>
         <!-- <box size="0.01 0.01 0.01" /> -->
-        <mesh filename="package://armada_description/armada_tooling/meshes/d435_mount_link.dae" />
+        <mesh filename="package://armada_description/armada_tooling/meshes/d435_mount_link.STL"/>
       </geometry>
     </collision>
@@ -66,5 +66,5 @@
       <geometry>
         <!-- <box size="0.01 0.01 0.01" /> -->
-        <mesh filename="package://armada_description/armada_tooling/meshes/d435.dae" />
+        <mesh filename="package://armada_description/armada_tooling/meshes/d435.STL"/>
       </geometry>
     </collision>
@@ -108,5 +108,5 @@
       <geometry>
         <!-- <box size="0.01 0.01 0.01" /> -->
-        <mesh filename="package://armada_description/armada_tooling/meshes/millibar_adapters_link.dae" />
+        <mesh filename="package://armada_description/armada_tooling/meshes/millibar_adapters_link.STL"/>
       </geometry>
     </collision>
@@ -138,5 +138,5 @@
       <geometry>
         <!-- <box size="0.01 0.01 0.01" /> -->
-        <mesh filename="package://armada_description/armada_tooling/meshes/r85_network_adapter_link.dae" />
+        <mesh filename="package://armada_description/armada_tooling/meshes/r85_network_adapter_link.STL"/>
       </geometry>
     </collision>

Commit message: add <realsense camera>_link which needs to be further parameterized to URDF for accurate transforms without static tf publisher, camera link name is defined by camera name parameter in camera bringup

File: armada_description/armada_tooling/urdf/d435_millibar_model_macro.urdf.xacro (robot description, xacro)
@@ -76,4 +76,18 @@
     <axis xyz="0 0 0" />
   </joint>
+  <!-- THIS IS THE EXPERIMENTAL CAMERA WRIST BIT -->
+  <!-- THIS IS THE EXPERIMENTAL CAMERA WRIST BIT -->
+  <!-- THIS IS THE EXPERIMENTAL CAMERA WRIST BIT -->
+  <!-- THIS IS THE EXPERIMENTAL CAMERA WRIST BIT -->
+  <link name="camera_wrist_link"/>
+  <joint name="${prefix}d435_to_camera_wrist_joint" type="fixed">
+    <parent link="${prefix}d435"/>
+    <child link="${prefix}camera_wrist_link"/>
+    <origin xyz="0.0175 0.0 0.025" rpy="0.0 -${pi/2} -${pi/2}"/>
+   </joint>
+   <!-- THIS IS THE EXPERIMENTAL CAMERA WRIST BIT -->
+   <!-- THIS IS THE EXPERIMENTAL CAMERA WRIST BIT -->
+   <!-- THIS IS THE EXPERIMENTAL CAMERA WRIST BIT -->
+   <!-- THIS IS THE EXPERIMENTAL CAMERA WRIST BIT -->
   <link name="${prefix}d435_inter_link" />
   <joint name="${prefix}d435_to_d435_inter_joint" type="fixed">

Commit message: remove dummy tcp link; manipulator chain now references tool_frame defined in gripper urdf

File: armada_description/armada_tooling/urdf/d435_millibar_model_macro.urdf.xacro (robot description, xacro)
@@ -171,12 +171,4 @@
     <axis xyz="0 0 0" />
   </joint>
-  <!-- dummy tcp_link for controlling -->
-  <link name="${prefix}tcp_link"/>
-  <joint name="${prefix}tcpip_adapter_to_tcp_joint" type="fixed">
-    <origin xyz="0.0 0.0 0.14" rpy="0 0 0" />
-    <parent link="${prefix}r85_network_adapter_link" />
-    <child link="${prefix}tcp_link" />
-    <axis xyz="0 0 0" />
-  </joint>
   </xacro:macro>
 </robot>

Commit message: remove old comments/notes, unused taglines/macros, add prefix tag to untagged component

File: armada_description/armada_tooling/urdf/d435_millibar_model_macro.urdf.xacro (robot description, xacro)
@@ -14,8 +14,5 @@
     xmlns:xacro="http://ros.org/wiki/xacro">
   <xacro:macro name="d435_millibar" params="prefix parent">
-  <!-- add in a namespace param and update lines 82/83 & 89/90 where a namespace would be used for wrist cam -->
-  <xacro:include filename="$(find armada_gazebo)/armada_tooling/urdf/d435_millibar_model_gazebo.xacro" />
   <xacro:include filename="$(find armada_gazebo)/armada_tooling/urdf/d435_millibar_depth_camera_gazebo.xacro" />
-  <xacro:d435_millibar_gazebo prefix="${prefix}" />
   <xacro:d435_millibar_depth_camera_gazebo prefix="${prefix}" />
   <link name="${prefix}d435_mount_link">
@@ -37,5 +34,4 @@
       <origin xyz="0 0 0" rpy="0 0 0" />
       <geometry>
-        <!-- <box size="0.01 0.01 0.01" /> -->
         <mesh filename="package://armada_description/armada_tooling/meshes/d435_mount_link.STL"/>
       </geometry>
@@ -65,5 +61,4 @@
       <origin xyz="0 0 0" rpy="0 0 0" />
       <geometry>
-        <!-- <box size="0.01 0.01 0.01" /> -->
         <mesh filename="package://armada_description/armada_tooling/meshes/d435.STL"/>
       </geometry>
@@ -76,9 +71,5 @@
     <axis xyz="0 0 0" />
   </joint>
-  <!-- THIS IS THE EXPERIMENTAL CAMERA WRIST BIT -->
-  <!-- THIS IS THE EXPERIMENTAL CAMERA WRIST BIT -->
-  <!-- THIS IS THE EXPERIMENTAL CAMERA WRIST BIT -->
-  <!-- THIS IS THE EXPERIMENTAL CAMERA WRIST BIT -->
-  <link name="camera_wrist_link"/>
+  <link name="${prefix}camera_wrist_link"/>
   <joint name="${prefix}d435_to_camera_wrist_joint" type="fixed">
     <parent link="${prefix}d435"/>
@@ -86,8 +77,4 @@
     <origin xyz="0.0175 0.0 0.025" rpy="0.0 -${pi/2} -${pi/2}"/>
    </joint>
-   <!-- THIS IS THE EXPERIMENTAL CAMERA WRIST BIT -->
-   <!-- THIS IS THE EXPERIMENTAL CAMERA WRIST BIT -->
-   <!-- THIS IS THE EXPERIMENTAL CAMERA WRIST BIT -->
-   <!-- THIS IS THE EXPERIMENTAL CAMERA WRIST BIT -->
   <link name="${prefix}d435_inter_link" />
   <joint name="${prefix}d435_to_d435_inter_joint" type="fixed">
